File: EloadV2/ELoad.kicad_sch (KiCad schematic)
At the start: 107 parts, among them J1 Power Input, J2 Conn_01x02, J3 OLED, J4 ENCODER, J5 SWDEBUG, M1 Fan_4pin, Q4 Q_NMOS_GDS, U1 TL072, U10 TL072, U11 LTV-817S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

Commit message: removing power, waveform generation, op amp pi, button latch
Parts:
- removed C1: 10u, Capacitor_SMD:C_1206_3216Metric_Pad1.33x1.80mm_HandSolder, symbol Device:C_Small
- removed C18, C7: 0.1u, Capacitor_SMD:C_0603_1608Metric_Pad1.08x0.95mm_HandSolder, symbol Device:C_Small
- removed C2, C25: 10u, Capacitor_SMD:C_0603_1608Metric_Pad1.08x0.95mm_HandSolder, symbol Device:C_Small
- removed C26, C4, C8, C9: 22u, Capacitor_SMD:C_0603_1608Metric_Pad1.08x0.95mm_HandSolder, symbol Device:C_Small
- removed C5: 100n, Capacitor_SMD:C_0603_1608Metric_Pad1.08x0.95mm_HandSolder, symbol Device:C_Small
- removed C6: 1u, Capacitor_SMD:C_0603_1608Metric_Pad1.08x0.95mm_HandSolder, symbol Device:C_Small
- removed C?: 0.01u, Capacitor_SMD:C_0603_1608Metric_Pad1.08x0.95mm_HandSolder, symbol Device:C_Small
- removed C?: 0.001u, Capacitor_SMD:C_0603_1608Metric_Pad1.08x0.95mm_HandSolder, symbol Device:C_Small
- removed J4: ENCODER, Connector_PinSocket_2.54mm:PinSocket_1x06_P2.54mm_Vertical, symbol Connector_Generic:Conn_01x06
- removed L1: 2.2u, Inductor_SMD:L_1008_2520Metric_Pad1.43x2.20mm_HandSolder, symbol Device:L_Small
- removed R1: 70k, Resistor_SMD:R_0805_2012Metric_Pad1.20x1.40mm_HandSolder, symbol Device:R_Small
- removed R10, R11, R12, R19, R2, R21, R23, R3, R6, R8, R9, R? (x2): 10k, Resistor_SMD:R_0805_2012Metric_Pad1.20x1.40mm_HandSolder, symbol Device:R_Small
- removed R13, R5, R? (x2): 100, Resistor_SMD:R_0805_2012Metric_Pad1.20x1.40mm_HandSolder, symbol Device:R_Small
- removed R14, R24: 3.3k, Resistor_SMD:R_0805_2012Metric_Pad1.20x1.40mm_HandSolder, symbol Device:R_Small
- removed R15: 60k, Resistor_SMD:R_0805_2012Metric_Pad1.20x1.40mm_HandSolder, symbol Device:R_Small
- removed R16: 4k, Resistor_SMD:R_0805_2012Metric_Pad1.20x1.40mm_HandSolder, symbol Device:R_Small
- removed R18: 52.3k, Resistor_SMD:R_0805_2012Metric_Pad1.20x1.40mm_HandSolder, symbol Device:R_Small
- removed R22, R4: 1.7k, Resistor_SMD:R_0805_2012Metric_Pad1.20x1.40mm_HandSolder, symbol Device:R_Small
- removed R?: 110.42, Resistor_SMD:R_0805_2012Metric_Pad1.20x1.40mm_HandSolder, symbol Device:R_Small
- removed R?: 4.3k, Resistor_SMD:R_0805_2012Metric_Pad1.20x1.40mm_HandSolder, symbol Device:R_Small
- removed R?: 2k, Resistor_SMD:R_0805_2012Metric_Pad1.20x1.40mm_HandSolder, symbol Device:R_Small
- removed R?: 4480, Resistor_SMD:R_0805_2012Metric_Pad1.20x1.40mm_HandSolder, symbol Device:R_Small
- removed TP1, TP10, TP3, TP4, TP6: TestPoint_Probe, TestPoint:TestPoint_Pad_1.5x1.5mm, symbol Connector:TestPoint_Probe
- removed TP2, TP5: Test, TestPoint:TestPoint_Pad_1.5x1.5mm, symbol Connector:TestPoint_Probe
- removed U1, U10, U14, U5: TL072, Package_SO:SOIC-8_3.9x4.9mm_P1.27mm, symbol Amplifier_Operational:TL072
- removed U13: AZ1117-5.0, Package_TO_SOT_SMD:SOT-223-3_TabPin2, symbol Regulator_Linear:AZ1117-5.0
- removed U15: MCP9700AT-ETT, Package_TO_SOT_THT:TO-92, symbol Sensor_Temperature:MCP9700AT-ETT
- removed U2: AZ1117-3.3, Package_TO_SOT_SMD:SOT-89-3_Handsoldering, symbol Regulator_Linear:AZ1117-3.3
- removed U4: AP62250WU-7, Package_TO_SOT_SMD:TSOT-23-6, symbol Regulator_Switching:AP62250WU-7
- removed U6: TL074, Package_SO:SOIC-14_3.9x8.7mm_P1.27mm, symbol Amplifier_Operational:TL074
- removed unit 3 of U8
- removed U9: LM393, Package_SO:SOIC-8_3.9x4.9mm_P1.27mm, symbol Comparator:LM393
- removed U?: NE555D, Package_SO:SOIC-8_3.9x4.9mm_P1.27mm, symbol Timer:NE555D
- removed U?: TL072, symbol Amplifier_Operational:TL072
- removed X1: ECS-2520MV-160-CN-TR, Oscillator:Oscillator_SMD_ECS_2520MV-xxx-xx-4Pin_2.5x2.0mm, symbol Oscillator:ECS-2520MV-xxx-xx
Connections:
- net +5V is gone; now on net +3V3: C3.2, U3.4 (Vdd)
- net ROT_CCW: no longer names the net of U12.15 (PA5)
- net ROT_CW: no longer names the net of U12.11 (PA1)
- no-connect marks 45 -> 32
Other:
- note removed: "16kHz Triangle Wave"
- note removed: "70k out of stock r15, r1 = 56k r11,r2 = 8k"
- note removed: "PI"
- note removed: "Temperature"
- moved on the sheet: U8B
